File: datakeyboard/datakeyboard.kicad_sch (KiCad schematic)
At the start: 42 parts, among them Q1 BSS83P, Q2 BSS83P, Q3 BSS83P, SW1 SW_Push, SW2 SW_Push, SW3 SW_Push, SW4 SW_Push, SW5 SW_Push, SW6 SW_Push, U1 PIC24FJ128GB204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

Commit message: Start board layout
Parts:
- JBAT1, JCASE1: footprint Connector_PinHeader_2.54mm:PinHeader_1x02_P2.54mm_Vertical -> Resistor_SMD:R_1206_3216Metric_Pad1.30x1.75mm_HandSolder
- JCARD1: footprint Connector_Card:microSD_HC_Hirose_DM3AT-SF-PEJM5 -> Library:microSD_Unknown
- JUSB1: footprint Connector_USB:USB_Micro-B_Molex-105017-0001 -> Library:USB_Micro-B_Unknown
Connections:
- net SDCard_CD: now also JCARD1.9 (DET_B); no longer JCARD1.10 (DET_A)
- no-connect marks 10 -> 11
Changed lines of the file:
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@@
   (no_connect (at 132.08 90.17))
   (no_connect (at 175.26 135.89))
-  (no_connect (at 227.33 60.96))
+  (no_connect (at 158.75 27.94))
+  (no_connect (at 227.33 58.42))
   (wire (pts (xy 213.36 107.95) (xy 212.09 107.95))
     (stroke (width 0) (type default) (color 0 0 0 0))
@@
     (stroke (width 0) (type default) (color 0 0 0 0))
   )
-  (wire (pts (xy 217.17 58.42) (xy 227.33 58.42))
+  (wire (pts (xy 217.17 60.96) (xy 227.33 60.96))
     (stroke (width 0) (type default) (color 0 0 0 0))
   )
@@
     (effects (font (size 1.27 1.27)) (justify right bottom))
   )
-  (label "SDCard_CD" (at 217.17 58.42 0)
+  (label "SDCard_CD" (at 217.17 60.96 0)
     (effects (font (size 1.27 1.27)) (justify left bottom))
   )
@@
     (property "Reference" "JCARD1" (id 0) (at 250.825 26.67 0))
     (property "Value" "Micro_SD_Card_Det" (id 1) (at 250.825 29.21 0))
-    (property "Footprint" "Connector_Card:microSD_HC_Hirose_DM3AT-SF-PEJM5" (id 2) (at 302.26 30.48 0)
+    (property "Footprint" "Library:microSD_Unknown" (id 2) (at 302.26 30.48 0)
       (effects (font (size 1.27 1.27)) hide)
     )
@@
       (effects (font (size 1.27 1.27)) (justify right))
     )
-    (property "Footprint" "Connector_PinHeader_2.54mm:PinHeader_1x02_P2.54mm_Vertical" (id 2) (at 144.78 21.59 0)
+    (property "Footprint" "Resistor_SMD:R_1206_3216Metric_Pad1.30x1.75mm_HandSolder" (id 2) (at 144.78 21.59 0)
       (effects (font (size 1.27 1.27)) hide)
     )
@@
       (effects (font (size 1.27 1.27)) (justify right))
     )
-    (property "Footprint" "Connector_PinHeader_2.54mm:PinHeader_1x02_P2.54mm_Vertical" (id 2) (at 88.9 21.59 0)
+    (property "Footprint" "Resistor_SMD:R_1206_3216Metric_Pad1.30x1.75mm_HandSolder" (id 2) (at 88.9 21.59 0)
       (effects (font (size 1.27 1.27)) hide)
     )
@@
     (property "Reference" "JUSB1" (id 0) (at 48.26 82.55 0))
     (property "Value" "USB_OTG" (id 1) (at 48.26 85.09 0))
-    (property "Footprint" "Connector_USB:USB_Micro-B_Molex-105017-0001" (id 2) (at 52.07 96.52 0)
+    (property "Footprint" "Library:USB_Micro-B_Unknown" (id 2) (at 52.07 96.52 0)
       (effects (font (size 1.27 1.27)) hide)
     )
@@
     )
     (path "/a3fb3ec1-d439-4e28-9c23-0b3ef6bab1e5"
-      (reference "JBAT1") (unit 1) (value "Conn_01x02") (footprint "Connector_PinHeader_2.54mm:PinHeader_1x02_P2.54mm_Vertical")
+      (reference "JBAT1") (unit 1) (value "Conn_01x02") (footprint "Resistor_SMD:R_1206_3216Metric_Pad1.30x1.75mm_HandSolder")
     )
     (path "/736d6c1c-614a-4b0f-8fe3-6b0669b7a1b9"
-      (reference "JCARD1") (unit 1) (value "Micro_SD_Card_Det") (footprint "Connector_Card:microSD_HC_Hirose_DM3AT-SF-PEJM5")
+      (reference "JCARD1") (unit 1) (value "Micro_SD_Card_Det") (footprint "Library:microSD_Unknown")
     )
     (path "/a0d77163-a822-4f35-a314-d39c42d23672"
-      (reference "JCASE1") (unit 1) (value "Conn_01x02") (footprint "Connector_PinHeader_2.54mm:PinHeader_1x02_P2.54mm_Vertical")
+      (reference "JCASE1") (unit 1) (value "Conn_01x02") (footprint "Resistor_SMD:R_1206_3216Metric_Pad1.30x1.75mm_HandSolder")
     )
     (path "/d37334a6-f13d-49cb-afe8-430745ecfc0f"
@@
     )
     (path "/e1976fd7-61fd-44d2-a0bf-7b78c6303643"
-      (reference "JUSB1") (unit 1) (value "USB_OTG") (footprint "Connector_USB:USB_Micro-B_Molex-105017-0001")
+      (reference "JUSB1") (unit 1) (value "USB_OTG") (footprint "Library:USB_Micro-B_Unknown")
     )
     (path "/14f0f55b-770f-492a-a96d-c71bf97952d8"

Commit message: Finish PCB layout
Connections:
- net BNT4 is gone; now on net BTN4: SW4.2
- net GND: no longer U1.34 (RA4)
- net CHRG: now reaches R2.2, U2.7 (CHRG)
- net CHRG: now also U1.34 (RA4)
- no-connect marks 11 -> 10
Changed lines of the file:
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@@
   (no_connect (at 132.08 90.17))
   (no_connect (at 175.26 135.89))
-  (no_connect (at 158.75 27.94))
   (no_connect (at 227.33 58.42))
   (wire (pts (xy 213.36 107.95) (xy 212.09 107.95))
@@
     (stroke (width 0) (type default) (color 0 0 0 0))
   )
-  (wire (pts (xy 167.64 64.77) (xy 167.64 67.31))
+  (wire (pts (xy 167.64 57.15) (xy 167.64 67.31))
     (stroke (width 0) (type default) (color 0 0 0 0))
   )
@@
     (stroke (width 0) (type default) (color 0 0 0 0))
   )
+  (wire (pts (xy 88.9 26.67) (xy 88.9 50.8))
+    (stroke (width 0) (type default) (color 0 0 0 0))
+  )
   (wire (pts (xy 245.11 86.36) (xy 245.11 101.6))
     (stroke (width 0) (type default) (color 0 0 0 0))
@@
   )
   (wire (pts (xy 201.93 88.9) (xy 201.93 100.33))
-    (stroke (width 0) (type default) (color 0 0 0 0))
-  )
-  (wire (pts (xy 88.9 26.67) (xy 88.9 50.8))
     (stroke (width 0) (type default) (color 0 0 0 0))
   )
@@
     (effects (font (size 1.27 1.27)) (justify right bottom))
   )
+  (label "CHRG" (at 167.64 57.15 270)
+    (effects (font (size 1.27 1.27)) (justify right bottom))
+  )
   (label "MOSI" (at 217.17 43.18 0)
     (effects (font (size 1.27 1.27)) (justify left bottom))
@@
     (effects (font (size 1.27 1.27)) (justify left bottom))
   )
+  (label "CHRG" (at 58.42 45.72 0)
+    (effects (font (size 1.27 1.27)) (justify left bottom))
+  )
   (label "RES_D" (at 252.73 92.71 90)
     (effects (font (size 1.27 1.27)) (justify left bottom))
@@
     (effects (font (size 1.27 1.27)) (justify left bottom))
   )
-  (label "BNT4" (at 215.9 154.94 180)
+  (label "BTN4" (at 215.9 154.94 180)
     (effects (font (size 1.27 1.27)) (justify right bottom))
   )
@@
     (pin "1")
     (pin "2")
-  )
-  (symbol (lib_id "power:GND") (at 167.64 64.77 180) (unit 1)
-    (in_bom yes) (on_board yes) (fields_autoplaced)
-    (property "Reference" "#PWR0103" (id 0) (at 167.64 58.42 0)
-      (effects (font (size 1.27 1.27)) hide)
-    )
-    (property "Value" "GND" (id 1) (at 167.64 59.69 0))
-    (property "Footprint" "" (id 2) (at 167.64 64.77 0)
-      (effects (font (size 1.27 1.27)) hide)
-    )
-    (property "Datasheet" "" (id 3) (at 167.64 64.77 0)
-      (effects (font (size 1.27 1.27)) hide)
-    )
-    (pin "1")
   )
   (symbol (lib_id "Device:C_Small") (at 27.94 176.53 0) (unit 1)
@@
       (reference "#PWR0102") (unit 1) (value "GND") (footprint "")
     )
-    (path "/300e80f5-a4d8-4fe2-b3c8-d2290a7011ab"
-      (reference "#PWR0103") (unit 1) (value "GND") (footprint "")
-    )
     (path "/de3db794-220c-46f9-91bf-bef667b33487"

Commit message: Add second regulator to bypass charger
Parts:
- removed U2: TP4056, Package_SO:SO-8_5.3x6.2mm_P1.27mm, symbol Library:TP4056
- added U2: MCP73831-2-OT, Package_TO_SOT_SMD:SOT-23-5, symbol Battery_Management:MCP73831-2-OT
- added U4: STLQ015M33R, Package_TO_SOT_SMD:SOT-23-5, symbol Regulator_Linear:AP131-30
- C4: value 100nF -> 10uF; footprint Capacitor_SMD:C_0603_1608Metric_Pad1.08x0.95mm_HandSolder -> Capacitor_SMD:C_0805_2012Metric_Pad1.18x1.45mm_HandSolder
- U3: value MIC5501-30 -> STLQ015M30R
Connections:
- net +3V0: now also U4.5 (OUT)
- net CHRG: now also U2.1 (STAT)
- net GND: now also C4.2, JCARD1.10 (DET_A), R3.2, U2.2 (VSS), U4.2 (GND); no longer C4.1
- net VBAT: now also U2.3 (VBAT)
- net VUSB: now also C4.1, U2.4 (VDD), U4.1 (IN), U4.3 (EN); no longer C4.2
- net at R9.2: now also U2.5 (PROG)
Other:
- moved on the sheet: C2, R9, U3

Commit message: Control charging by microcontroller
Parts:
- added Q4: BSS83P, Package_TO_SOT_SMD:SOT-23, symbol Transistor_FET:BSS83P
- added R12: 10k, Resistor_SMD:R_0805_2012Metric_Pad1.20x1.40mm_HandSolder, symbol Device:R_Small
Connections:
- net VUSB: now also Q4.2 (S), R12.1; no longer U2.4 (VDD)
- net CHRG_PWR: now reaches U1.36 (RC3)
- net CHRG_PWR: now also Q4.1 (G), R12.2
- new net: Q4.3 (D), U2.4 (VDD)
- no-connect marks 10 -> 9
Changed lines of the file:
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@@
   (junction (at 119.38 66.04) (diameter 0) (color 0 0 0 0)
   )
+  (junction (at 33.02 22.86) (diameter 0) (color 0 0 0 0)
+  )
   (junction (at 27.94 173.99) (diameter 0) (color 0 0 0 0)
   )
   (junction (at 212.09 88.9) (diameter 0) (color 0 0 0 0)
   )
+  (junction (at 25.4 29.21) (diameter 0) (color 0 0 0 0)
+  )
   (junction (at 57.15 68.58) (diameter 0) (color 0 0 0 0)
   )
@@
   (junction (at 33.02 62.23) (diameter 0) (color 0 0 0 0)
   )
+  (junction (at 57.15 22.86) (diameter 0) (color 0 0 0 0)
+  )
   (junction (at 64.77 22.86) (diameter 0) (color 0 0 0 0)
   )
   (junction (at 236.22 96.52) (diameter 0) (color 0 0 0 0)
   )
-  (junction (at 57.15 35.56) (diameter 0) (color 0 0 0 0)
-  )
   (junction (at 97.79 38.1) (diameter 0) (color 0 0 0 0)
   )
@@
   )
   (no_connect (at 114.3 38.1))
-  (no_connect (at 162.56 67.31))
   (no_connect (at 227.33 55.88))
   (no_connect (at 227.33 38.1))
@@
     (stroke (width 0) (type default) (color 0 0 0 0))
   )
+  (wire (pts (xy 31.75 22.86) (xy 33.02 22.86))
+    (stroke (width 0) (type default) (color 0 0 0 0))
+  )
   (wire (pts (xy 218.44 82.55) (xy 222.25 82.55))
     (stroke (width 0) (type default) (color 0 0 0 0))
@@
     (stroke (width 0) (type default) (color 0 0 0 0))
   )
+  (wire (pts (xy 25.4 22.86) (xy 25.4 29.21))
+    (stroke (width 0) (type default) (color 0 0 0 0))
+  )
   (wire (pts (xy 45.72 105.41) (xy 45.72 107.95))
     (stroke (width 0) (type default) (color 0 0 0 0))
@@
     (stroke (width 0) (type default) (color 0 0 0 0))
   )
-  (wire (pts (xy 57.15 35.56) (xy 57.15 22.86))
-    (stroke (width 0) (type default) (color 0 0 0 0))
-  )
   (wire (pts (xy 96.52 132.08) (xy 96.52 133.35))
     (stroke (width 0) (type default) (color 0 0 0 0))
@@
     (stroke (width 0) (type default) (color 0 0 0 0))
   )
-  (wire (pts (xy 57.15 35.56) (xy 57.15 68.58))
+  (wire (pts (xy 57.15 22.86) (xy 57.15 68.58))
     (stroke (width 0) (type default) (color 0 0 0 0))
   )
@@
     (stroke (width 0) (type default) (color 0 0 0 0))
   )
+  (wire (pts (xy 33.02 22.86) (xy 33.02 24.13))
+    (stroke (width 0) (type default) (color 0 0 0 0))
+  )
   (wire (pts (xy 177.8 97.79) (xy 187.96 97.79))
     (stroke (width 0) (type default) (color 0 0 0 0))
@@
     (stroke (width 0) (type default) (color 0 0 0 0))
   )
+  (wire (pts (xy 13.97 29.21) (xy 25.4 29.21))
+    (stroke (width 0) (type default) (color 0 0 0 0))
+  )
   (wire (pts (xy 62.23 173.99) (xy 73.66 173.99))
     (stroke (width 0) (type default) (color 0 0 0 0))
@@
     (stroke (width 0) (type default) (color 0 0 0 0))
   )
+  (wire (pts (xy 33.02 22.86) (xy 57.15 22.86))
+    (stroke (width 0) (type default) (color 0 0 0 0))
+  )
   (wire (pts (xy 76.2 33.02) (xy 76.2 35.56))
     (stroke (width 0) (type default) (color 0 0 0 0))
@@
     (stroke (width 0) (type default) (color 0 0 0 0))
   )
+  (wire (pts (xy 162.56 52.07) (xy 162.56 67.31))
+    (stroke (width 0) (type default) (color 0 0 0 0))
+  )
   (wire (pts (xy 88.9 76.2) (xy 88.9 78.74))
     (stroke (width 0) (type default) (color 0 0 0 0))
@@
     (stroke (width 0) (type default) (color 0 0 0 0))
   )
-  (wire (pts (xy 33.02 35.56) (xy 57.15 35.56))
-    (stroke (width 0) (type default) (color 0 0 0 0))
-  )
   (wire (pts (xy 242.57 86.36) (xy 242.57 91.44))
     (stroke (width 0) (type default) (color 0 0 0 0))
@@
     (stroke (width 0) (type default) (color 0 0 0 0))
   )
+  (wire (pts (xy 26.67 22.86) (xy 25.4 22.86))
+    (stroke (width 0) (type default) (color 0 0 0 0))
+  )
   (wire (pts (xy 73.66 173.99) (xy 85.09 173.99))
     (stroke (width 0) (type default) (color 0 0 0 0))
@@
     (stroke (width 0) (type default) (color 0 0 0 0))
   )
-  (wire (pts (xy 33.02 45.72) (xy 33.02 35.56))
+  (wire (pts (xy 33.02 34.29) (xy 33.02 45.72))
     (stroke (width 0) (type default) (color 0 0 0 0))
   )
@@
     (effects (font (size 1.27 1.27)) (justify right bottom))
   )
+  (label "CHRG_PWR" (at 13.97 29.21 0)
+    (effects (font (size 1.27 1.27)) (justify left bottom))
+  )
   (label "MOSI" (at 125.73 82.55 0)
     (effects (font (size 1.27 1.27)) (justify left bottom))
@@
   (label "RES_D" (at 252.73 92.71 90)
     (effects (font (size 1.27 1.27)) (justify left bottom))
+  )
+  (label "CHRG_PWR" (at 162.56 52.07 270)
+    (effects (font (size 1.27 1.27)) (justify right bottom))
   )
   (label "VOLT_PWR" (at 109.22 120.65 0)
@@
     (pin "2")
   )
+  (symbol (lib_id "Device:R_Small") (at 29.21 22.86 270) (unit 1)
+    (in_bom yes) (on_board yes) (fields_autoplaced)
+    (property "Reference" "R12" (id 0) (at 29.21 16.51 90))
+    (property "Value" "10k" (id 1) (at 29.21 19.05 90))
+    (property "Footprint" "Resistor_SMD:R_0805_2012Metric_Pad1.20x1.40mm_HandSolder" (id 2) (at 29.21 22.86 0)
+      (effects (font (size 1.27 1.27)) hide)
+    )
+    (property "Datasheet" "~" (id 3) (at 29.21 22.86 0)
+      (effects (font (size 1.27 1.27)) hide)
+    )
+    (pin "1")
+    (pin "2")
+  )
   (symbol (lib_id "Switch:SW_Push") (at 207.01 139.7 0) (unit 1)
     (in_bom yes) (on_board yes) (fields_autoplaced)
@@
     )
     (pin "1")
+  )
+  (symbol (lib_id "Transistor_FET:BSS83P") (at 30.48 29.21 0) (mirror x) (unit 1)
+    (in_bom yes) (on_board yes) (fields_autoplaced)
+    (property "Reference" "Q4" (id 0) (at 36.83 27.9399 0)
+      (effects (font (size 1.27 1.27)) (justify left))
+    )
+    (property "Value" "BSS83P" (id 1) (at 36.83 30.4799 0)
+      (effects (font (size 1.27 1.27)) (justify left))
+    )
+    (property "Footprint" "Package_TO_SOT_SMD:SOT-23" (id 2) (at 35.56 27.305 0)
+      (effects (font (size 1.27 1.27) italic) (justify left) hide)
+    )
+    (property "Datasheet" "http://www.farnell.com/datasheets/1835997.pdf" (id 3) (at 30.48 29.21 0)
+      (effects (font (size 1.27 1.27)) (justify left) hide)
+    )
+    (pin "1")
+    (pin "2")
+    (pin "3")
   )
   (symbol (lib_id "power:GND") (at 27.94 180.34 0) (unit 1)
@@
   (symbol (lib_id "power:GND") (at 217.17 58.42 270) (unit 1)
     (in_bom yes) (on_board yes) (fields_autoplaced)
-    (property "Reference" "#PWR?" (id 0) (at 210.82 58.42 0)
+    (property "Reference" "#PWR01" (id 0) (at 210.82 58.42 0)
       (effects (font (size 1.27 1.27)) hide)
     )
@@
   )
   (symbol_instances
+    (path "/a1205476-90dd-410e-9d3f-9e2a8ef17be6"
+      (reference "#PWR01") (unit 1) (value "GND") (footprint "")
+    )
     (path "/71f64ba2-8ec2-46c9-b279-dafa59091949"
       (reference "#PWR02") (unit 1) (value "+3V0") (footprint "")
@@
       (reference "#PWR0111") (unit 1) (value "GND") (footprint "")
     )
-    (path "/a1205476-90dd-410e-9d3f-9e2a8ef17be6"
-      (reference "#PWR?") (unit 1) (value "GND") (footprint "")
-    )
     (path "/c9228fbc-419a-427a-86c6-4b3d3b0ccaea"
       (reference "C1") (unit 1) (value "10uF") (footprint "Capacitor_SMD:C_0805_2012Metric_Pad1.18x1.45mm_HandSolder")
@@
       (reference "Q3") (unit 1) (value "BSS83P") (footprint "Package_TO_SOT_SMD:SOT-23")
     )
+    (path "/0e8e948e-2b60-41cb-ae6a-54a151f21e4d"
+      (reference "Q4") (unit 1) (value "BSS83P") (footprint "Package_TO_SOT_SMD:SOT-23")
+    )
     (path "/f5dfac85-0fba-4fec-986d-820052834f83"
       (reference "R1") (unit 1) (value "100") (footprint "Resistor_SMD:R_0805_2012Metric_Pad1.20x1.40mm_HandSolder")
@@
       (reference "R11") (unit 1) (value "10k") (footprint "Resistor_SMD:R_0805_2012Metric_Pad1.20x1.40mm_HandSolder")
     )
+    (path "/02eba330-4894-4282-85e3-083927dccf68"
+      (reference "R12") (unit 1) (value "10k") (footprint "Resistor_SMD:R_0805_2012Metric_Pad1.20x1.40mm_HandSolder")
+    )
     (path "/064eada3-5eb6-40f4-8df6-485674836a12"
